Commit message: Added mapping to dashboard and tuned effective wheel seperation

File: ros2_ws/src/charlie_description/urdf/charlie.urdf.xacro (robot description, xacro)
@@ -152,5 +152,5 @@
     <parent link="base_link"/>
     <child link="laser_frame"/>
-    <origin xyz="${laser_x} ${laser_y} ${laser_z}" rpy="0 0 0"/>
+    <origin xyz="${laser_x} ${laser_y} ${laser_z}" rpy="0 0 3.14159"/>
   </joint>
   <!-- Camera frame.
